File: PCB Schemas/Remote Control V2/RemoteControl.sch (EAGLE design)
At the start: 23 parts, among them IC1 ATMEGA328-PU, Q1 16MHz

Commit message: Finalized V1 and V2 of remote control
Parts:
- removed LD1: (no value), led:DUOLED-RG-C
- removed S1, S2, S3: (no value), switch-omron:40-XX
- removed S4: TL39PO, switch:TL39PO
- removed SV1: (no value), con-lstb:MA04-1
- removed U$1: XBEE-1B1, Xbee:XBEE-1B1
- removed U$2: LE33, Regulator:LE33
- added BUT_A, BUT_B, BUT_C: (no value), switch-omron:40-XX
- added D1: 1N4148DO35-7, diode:1N4148DO35-7
- added PROG: (no value), con-lstb:MA04-1
- added R6: 330k, resistor:R-EU_0207/7
- added REG1: LE33, Regulator:LE33
- added ST: (no value), led:DUOLED-RG-C
- added XBEE: XBEE-1B1, Xbee:XBEE-1B1
- J1: device con-jack:DCJ0303 -> Connectors:DCJ0303
- R2: value (none) -> 100k; device pot:TRIM_EU-CA9V -> resistor:R-EU_0207/7
- R3: value 220 -> 330
Connections:
- removed net BLUE_BUTTON: IC1.D4, S3.P, S3.P1
- removed net GREEN_BUTTON: IC1.D3,INT1,PWM, S2.P, S2.P1
- removed net N$9: IC1.ADC0, R2.S
- removed net RED_BUTTON: IC1.D2,INT0, S1.P, S1.P1
- new net BAT: IC1.ADC0, R2.2, R6.1
- new net BUTTON_A: BUT_A.P, BUT_A.P1, IC1.D2,INT0
- new net BUTTON_B: BUT_B.P, BUT_B.P1, IC1.D3,INT1,PWM
- new net BUTTON_C: BUT_C.P, BUT_C.P1, IC1.D4
- net GND: now also BUT_A.S, BUT_A.S1, BUT_B.S, BUT_B.S1, BUT_C.S, BUT_C.S1, J1.2, J1.3, PROG.1, R2.1, REG1.GND, ST.C, XBEE.GND; no longer J1.1, LD1.C, R2.E, S1.S, S1.S1, S2.S, S2.S1, S3.S, S3.S1, SV1.1, U$1.GND, U$2.GND
- net GREEN_LED: now also IC1.D11,PWM,MOSI; no longer IC1.D10,PWM
- net N$11: now also ST.AR; no longer LD1.AR
- net N$12: now also ST.AG; no longer LD1.AG
- net N$3: now also C5.1, D1.C, REG1.VI; no longer J1.2, J1.3, S4.O
- net N$6: now also PROG.2; no longer SV1.2
- net RED_LED: now also IC1.D10,PWM; no longer IC1.D11,PWM,MOSI
- net RX: now also PROG.3; no longer SV1.3
- net TX: now also PROG.4; no longer SV1.4
- net VCC: now also REG1.VO, XBEE.VDD; no longer U$1.VDD, U$2.VO
- net VIN: now also D1.A, J1.1, R6.2; no longer C5.1, R2.A, S4.P, U$2.VI
- net XBEE_RX: now also IC1.D7, XBEE.DOUT; no longer IC1.D8, U$1.DOUT
- net XBEE_TX: now also IC1.D8, XBEE.DIN; no longer IC1.D7, U$1.DIN
Other:
- note added: "BATTERY SENSOR"
- note added: "BUTTONS"
- note added: "MICROCONTROLLER"
- note added: "POWER"
- note added: "STATUS LED"
- note added: "XBEE MODULE"
- moved on the sheet: C1, C2, C3, C4, C5, C6, IC1, J1, LED1, Q1, R1, R3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

Commit message: Revised PCB schemas for V1 and V2
Parts:
- J1: device Connectors:DCJ0303 -> Connectors:DC_JACKPTH
Changed lines of the file:
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@@
 <?xml version="1.0" encoding="utf-8"?>
 <!DOCTYPE eagle SYSTEM "eagle.dtd">
-<eagle version="6.6.0">
+<eagle version="7.1.0">
 <drawing>
 <settings>
@@
 <layer number="54" name="bGND_GNDA" color="1" fill="9" visible="no" active="no"/>
 <layer number="56" name="wert" color="7" fill="1" visible="no" active="no"/>
+<layer number="57" name="tCAD" color="7" fill="1" visible="no" active="no"/>
 <layer number="91" name="Nets" color="2" fill="1" visible="yes" active="yes"/>
 <layer number="92" name="Busses" color="1" fill="1" visible="yes" active="yes"/>
@@
 <layer number="108" name="tplace-old" color="10" fill="1" visible="yes" active="yes"/>
 <layer number="109" name="ref-old" color="11" fill="1" visible="yes" active="yes"/>
+<layer number="110" name="fp0" color="7" fill="1" visible="no" active="yes"/>
+<layer number="111" name="LPC17xx" color="7" fill="1" visible="no" active="yes"/>
+<layer number="112" name="tSilk" color="7" fill="1" visible="no" active="yes"/>
+<layer number="113" name="IDFDebug" color="4" fill="1" visible="no" active="yes"/>
 <layer number="116" name="Patch_BOT" color="9" fill="4" visible="yes" active="yes"/>
 <layer number="121" name="_tsilk" color="7" fill="1" visible="yes" active="yes"/>
 <layer number="122" name="_bsilk" color="7" fill="1" visible="yes" active="yes"/>
+<layer number="123" name="tTestmark" color="7" fill="1" visible="no" active="yes"/>
+<layer number="124" name="bTestmark" color="7" fill="1" visible="no" active="yes"/>
 <layer number="125" name="_tNames" color="7" fill="1" visible="yes" active="yes"/>
+<layer number="126" name="_bNames" color="7" fill="1" visible="no" active="yes"/>
+<layer number="127" name="_tValues" color="7" fill="1" visible="no" active="yes"/>
+<layer number="128" name="_bValues" color="7" fill="1" visible="no" active="yes"/>
+<layer number="131" name="tAdjust" color="7" fill="1" visible="no" active="yes"/>
+<layer number="132" name="bAdjust" color="7" fill="1" visible="no" active="yes"/>
 <layer number="144" name="Drill_legend" color="7" fill="1" visible="yes" active="yes"/>
+<layer number="150" name="Notes" color="7" fill="1" visible="no" active="yes"/>
 <layer number="151" name="HeatSink" color="7" fill="1" visible="yes" active="yes"/>
+<layer number="152" name="_bDocu" color="7" fill="1" visible="no" active="yes"/>
+<layer number="153" name="FabDoc1" color="7" fill="1" visible="no" active="yes"/>
+<layer number="154" name="FabDoc2" color="7" fill="1" visible="no" active="yes"/>
+<layer number="155" name="FabDoc3" color="7" fill="1" visible="no" active="yes"/>
 <layer number="199" name="Contour" color="7" fill="1" visible="yes" active="yes"/>
 <layer number="200" name="200bmp" color="1" fill="10" visible="yes" active="yes"/>
@@
 <layer number="223" name="223bmp" color="24" fill="1" visible="no" active="no"/>
 <layer number="224" name="224bmp" color="25" fill="1" visible="no" active="no"/>
+<layer number="248" name="Housing" color="7" fill="1" visible="no" active="yes"/>
+<layer number="249" name="Edge" color="7" fill="1" visible="no" active="yes"/>
 <layer number="250" name="Descript" color="3" fill="1" visible="no" active="no"/>
 <layer number="251" name="SMDround" color="12" fill="11" visible="no" active="no"/>
@@
 <part name="GND8" library="supply1" deviceset="GND" device=""/>
 <part name="REG1" library="Regulator" deviceset="LE33" device=""/>
-<part name="J1" library="Connectors" deviceset="DCJ0303" device=""/>
+<part name="J1" library="Connectors" deviceset="DC_JACK" device="PTH"/>
 <part name="GND9" library="supply1" deviceset="GND" device=""/>
 <part name="GND10" library="supply1" deviceset="GND" device=""/>
@@
 <instance part="GND8" gate="1" x="50.8" y="53.34"/>
 <instance part="REG1" gate="G$1" x="-55.88" y="68.58"/>
-<instance part="J1" gate="G$1" x="-93.98" y="71.12"/>
+<instance part="J1" gate="J$1" x="-93.98" y="71.12"/>
 <instance part="GND9" gate="1" x="-55.88" y="58.42"/>
 <instance part="GND10" gate="1" x="-83.82" y="58.42"/>
@@
 </segment>
 <segment>
-<pinref part="J1" gate="G$1" pin="2"/>
+<pinref part="J1" gate="J$1" pin="2"/>
 <pinref part="GND10" gate="1" pin="GND"/>
 <wire x1="-86.36" y1="71.12" x2="-83.82" y2="71.12" width="0.1524" layer="91"/>
 <wire x1="-83.82" y1="71.12" x2="-83.82" y2="68.58" width="0.1524" layer="91"/>
-<pinref part="J1" gate="G$1" pin="3"/>
+<pinref part="J1" gate="J$1" pin="3"/>
 <wire x1="-83.82" y1="68.58" x2="-83.82" y2="60.96" width="0.1524" layer="91"/>
 <wire x1="-86.36" y1="68.58" x2="-83.82" y2="68.58" width="0.1524" layer="91"/>
@@
 </segment>
 <segment>
-<pinref part="J1" gate="G$1" pin="1"/>
+<pinref part="J1" gate="J$1" pin="1"/>
 <pinref part="D1" gate="G$1" pin="A"/>
 <wire x1="-86.36" y1="73.66" x2="-81.28" y2="73.66" width="0.1524" layer="91"/>
